File: ECAD_main/ECAD_main.kicad_sch (KiCad schematic)
At the start: 0 parts

Commit message: wip
Parts:
- added C1: 4.7u/6.3V, Capacitor_SMD:C_0805_2012Metric_Pad1.18x1.45mm_HandSolder, symbol Device:C
- added C2, C3, C4, C5, C6, C7: 100n/6.3V, Capacitor_SMD:C_0402_1005Metric, symbol Device:C
- added C8, C9: 8p/50V, Capacitor_SMD:C_0603_1608Metric_Pad1.08x0.95mm_HandSolder, symbol Device:C
- added D1: BAT43W, Diode_SMD:D_SOD-123, symbol Device:D_Schottky
- added D2: FYLS-0603UGC, LED_SMD:LED_0603_1608Metric_Pad1.05x0.95mm_HandSolder, symbol Device:LED
- added D3: FYLS-0603URC, LED_SMD:LED_0603_1608Metric_Pad1.05x0.95mm_HandSolder, symbol Device:LED
- added FB1: BLM18PG330SN1D, Inductor_SMD:L_0603_1608Metric_Pad1.05x0.95mm_HandSolder, symbol Device:FerriteBead_Small
- added HU1: ~, zpc-lib:OZON_TECH_LOGO, symbol zpc-lib:LOGO
- added J1: DEBUG_01x04, Connector_PinHeader_2.54mm:PinHeader_1x04_P2.54mm_Vertical, symbol Connector_Generic:Conn_01x04
- added R1: 100k, Resistor_SMD:R_0603_1608Metric_Pad0.98x0.95mm_HandSolder, symbol Device:R
- added R2, R3: 680, Resistor_SMD:R_0603_1608Metric_Pad0.98x0.95mm_HandSolder, symbol Device:R
- added SW1: KLS7-TS6606-13.0, Button_Switch_THT:SW_PUSH_6mm_H4.3mm, symbol Switch:SW_Push
- added TP1, TP2: ~, TestPoint:TestPoint_Pad_D1.0mm, symbol Connector:TestPoint
- added U1: STM32F103C8T6, Package_QFP:LQFP-48_7x7mm_P0.5mm, symbol MCU_ST_STM32F1:STM32F103C8Tx
- added Y1: NX3225GD-8MHz, zpc-lib:NX3225GD, symbol Device:Crystal
Connections:
- new net: C7.2, SW1.2, U1.7 (NRST)
- new net: D1.2 (A), J1.1 (Pin_1)
- new net: C9.2, U1.6 (PD1), Y1.1
- new net: R1.2, U1.44 (BOOT0)
- new net: C8.2, U1.5 (PD0), Y1.2
- new net: D2.2 (A), R2.1
- new net: D3.2 (A), R3.1
- new net 3V3: D1.1 (K), FB1.1
- new net DGND: C1.2, C2.1, C3.1, C4.1, C5.1, C6.1, C7.1, C8.1, C9.1, D2.1 (K), D3.1 (K), J1.4 (Pin_4), R1.1, SW1.1, U1.23 (VSS), U1.35 (VSS), U1.47 (VSS), U1.8 (VSSA)
- new net LED_SMALL_ERROR: R3.2, U1.11 (PA1)
- new net LED_SMALL_OK: R2.2, U1.10 (PA0)
- new net MCU_SMALL_VDD: C1.1, C2.2, C3.2, C4.2, C5.2, C6.2, FB1.2, U1.1 (VBAT), U1.24 (VDD), U1.36 (VDD), U1.48 (VDD), U1.9 (VDDA)
- new net SWCLK_SMALL: J1.3 (Pin_3), U1.37 (PA14)
- new net SWDIO_SMALL: J1.2 (Pin_2), U1.34 (PA13)
- new net USB_DM_SMALL: TP1.1, U1.32 (PA11)
- new net USB_DP_SMALL: TP2.1, U1.33 (PA12)
- no-connect marks 0 -> 29
Other:
- added sheet power (power.kicad_sch)
- company: МГТУ им. Н.Э. Баумана -> (none)

Commit message: fixed
Other:
- sheet power renamed Power
- sheet Power: file power.kicad_sch -> Power.kicad_sch
Changed lines of the file:
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@@
 	)
 	(junction
-		(at 271.78 53.34)
-		(diameter 0)
-		(color 0 0 0 0)
-	)
-	(junction
 		(at 284.48 40.64)
 		(diameter 0)
@@
 	(wire
 		(pts
-			(xy 271.78 53.34) (xy 278.13 53.34)
+			(xy 267.97 53.34) (xy 278.13 53.34)
 		)
 		(stroke
@@
 	(wire
 		(pts
-			(xy 267.97 53.34) (xy 271.78 53.34)
-		)
-		(stroke
-			(width 0)
-			(type default)
-		)
-	)
-	(wire
-		(pts
 			(xy 290.83 53.34) (xy 284.48 53.34)
 		)
@@
 	)
 	(symbol
-		(lib_id "power:PWR_FLAG")
-		(at 271.78 53.34 180)
-		(unit 1)
-		(exclude_from_sim no)
-		(in_bom yes)
-		(on_board yes)
-		(dnp no)
-		(fields_autoplaced yes)
-		(property "Reference" "#FLG04"
-			(at 271.78 55.245 0)
-			(effects
-				(font
-					(size 1.27 1.27)
-				)
-				(hide yes)
-			)
-		)
-		(property "Value" "PWR_FLAG"
-			(at 271.78 58.42 0)
-			(effects
-				(font
-					(size 1.27 1.27)
-				)
-			)
-		)
-		(property "Footprint" ""
-			(at 271.78 53.34 0)
-			(effects
-				(font
-					(size 1.27 1.27)
-				)
-				(hide yes)
-			)
-		)
-		(property "Datasheet" "~"
-			(at 271.78 53.34 0)
-			(effects
-				(font
-					(size 1.27 1.27)
-				)
-				(hide yes)
-			)
-		)
-		(property "Description" "Special symbol for telling ERC where power comes from"
-			(at 271.78 53.34 0)
-			(effects
-				(font
-					(size 1.27 1.27)
-				)
-				(hide yes)
-			)
-		)
-		(pin "1"
-		)
-		(instances
-			(project ""
-				(path "/e9ffbb94-33e2-4158-ac4a-a33b17b122cf"
-					(reference "#FLG04")
-					(unit 1)
-				)
-			)
-		)
-	)
-	(symbol
 		(lib_id "Device:R")
 		(at 295.91 78.74 90)
@@
 			(color 0 0 0 0.0000)
 		)
-		(property "Sheetname" "power"
+		(property "Sheetname" "Power"
 			(at 292.1 175.8184 0)
 			(effects
@@
 			)
 		)
-		(property "Sheetfile" "power.kicad_sch"
+		(property "Sheetfile" "Power.kicad_sch"
 			(at 292.1 192.3546 0)
 			(effects
